Commit message: Simulation: Double Turtlebot3, can move pallets

File: catkin_workspace/src/amazon_robot_description/urdf/amazon_warehouse_robot.gazebo.xacro (robot description, xacro)
@@ -1,5 +1,5 @@
 <?xml version="1.0"?>
 <robot name="amazon_robot2_sim" xmlns:xacro="http://ros.org/wiki/xacro">
-  <xacro:arg name="laser_visual"  default="true"/>
+  <xacro:arg name="laser_visual"  default="false"/>
   <xacro:arg name="camera_visual" default="false"/>
   <xacro:arg name="imu_visual"    default="false"/>
@@ -8,6 +8,6 @@
   </gazebo>
   <gazebo reference="wheel_left_link">
-    <mu1>0.1</mu1>
-    <mu2>0.1</mu2>
+    <mu1>20</mu1>
+    <mu2>20</mu2>
     <kp>500000.0</kp>
     <kd>10.0</kd>
@@ -18,6 +18,6 @@
   </gazebo>
   <gazebo reference="wheel_right_link">
-    <mu1>0.1</mu1>
-    <mu2>0.1</mu2>
+    <mu1>20</mu1>
+    <mu2>20</mu2>
     <kp>500000.0</kp>
     <kd>10.0</kd>
@@ -28,6 +28,6 @@
   </gazebo>
   <gazebo reference="caster_back_right_link">
-    <mu1>0.1</mu1>
-    <mu2>0.1</mu2>
+    <mu1>20</mu1>
+    <mu2>20</mu2>
     <kp>1000000.0</kp>
     <kd>100.0</kd>
@@ -37,6 +37,6 @@
   </gazebo>
   <gazebo reference="caster_back_left_link">
-    <mu1>0.1</mu1>
-    <mu2>0.1</mu2>
+    <mu1>20</mu1>
+    <mu2>20</mu2>
     <kp>1000000.0</kp>
     <kd>100.0</kd>
@@ -45,11 +45,8 @@
     <material>Gazebo/FlatBlack</material>
   </gazebo>
-  <gazebo reference="top_lift">
-    <mu1>0.1</mu1>
-    <mu2>0.1</mu2>
+  <gazebo reference="platform_joint">
+    <mu1>20000</mu1>
+    <mu2>20000</mu2>
     <kp>1000000.0</kp>
-    <kd>100.0</kd>
-    <minDepth>0.001</minDepth>
-    <maxVel>1.0</maxVel>
     <material>Gazebo/FlatBlack</material>
   </gazebo>
@@ -76,8 +73,12 @@
       <leftJoint>wheel_left_joint</leftJoint>
       <rightJoint>wheel_right_joint</rightJoint>
-      <wheelSeparation>0.287</wheelSeparation>
-      <wheelDiameter>0.066</wheelDiameter>
-      <wheelAcceleration>1</wheelAcceleration>
-      <wheelTorque>10</wheelTorque>
+      <!--      <wheelSeparation>0.287</wheelSeparation>-->
+      <wheelSeparation>0.574</wheelSeparation>
+<!--      <wheelDiameter>0.066</wheelDiameter>-->
+      <wheelDiameter>0.144</wheelDiameter>
+      <wheelAcceleration>4</wheelAcceleration>
+<!--      <wheelAcceleration>1</wheelAcceleration>-->
+      <wheelTorque>50</wheelTorque>
+<!--      <wheelTorque>10</wheelTorque>-->
       <rosDebugLevel>na</rosDebugLevel>
     </plugin>

File: catkin_workspace/src/amazon_robot_description/urdf/amazon_warehouse_robot.transmission.xacro (robot description, xacro)
@@ -1,5 +1,5 @@
 <?xml version="1.0"?>
 <robot xmlns:xacro="http://www.ros.org/wiki/xacro">
-        <transmission type="transmission_interface/SimpleTransmission" name="lift_screw_trans">
+        <transmission name="lift_screw_trans">
             <actuator name="lift_screw_motor" >
                 <hardwareInterface>EffortJointInterface</hardwareInterface>
@@ -8,4 +8,5 @@
                 <hardwareInterface>EffortJointInterface</hardwareInterface>
             </joint>
+            <type>transmission_interface/SimpleTransmission</type>
             <mechanicalReduction>-47641.53</mechanicalReduction>
             <simulated_actuated_joint name="lift_screw_motor_screw_joint"

File: catkin_workspace/src/amazon_robot_description/urdf/amazon_warehouse_robot.urdf.xacro (robot description, xacro)
@@ -14,5 +14,5 @@
       <origin xyz="-0.064 0 0.0" rpy="0 0 0"/>
       <geometry>
-        <mesh filename="package://amazon_robot_description/meshes/bases/waffle_pi_base.stl" scale="0.001 0.001 0.001"/>
+        <mesh filename="package://amazon_robot_description/meshes/bases/waffle_pi_base.stl" scale="0.002 0.002 0.002"/>
       </geometry>
       <material name="orange"/>
@@ -21,5 +21,5 @@
       <origin xyz="-0.064 0 0.047" rpy="0 0 0"/>
       <geometry>
-        <box size="0.266 0.266 0.094"/>
+        <box size="0.532 0.532 0.188"/>
       </geometry>
     </collision>
@@ -35,5 +35,5 @@
     <parent link="base_link"/>
     <child link="wheel_left_link"/>
-    <origin xyz="0.0 0.144 0.023" rpy="-1.57 0 0"/>
+    <origin xyz="0.0 0.288 0.023" rpy="-1.57 0 0"/>
     <axis xyz="0 0 1"/>
   </joint>
@@ -42,5 +42,5 @@
       <origin xyz="0 0 0" rpy="1.57 0 0"/>
       <geometry>
-        <mesh filename="package://amazon_robot_description/meshes/wheels/left_tire.stl" scale="0.001 0.001 0.001"/>
+        <mesh filename="package://amazon_robot_description/meshes/wheels/left_tire.stl" scale="0.002 0.002 0.002"/>
       </geometry>
       <material name="dark"/>
@@ -49,5 +49,5 @@
       <origin xyz="0 0 0" rpy="0 0 0"/>
       <geometry>
-        <cylinder length="0.018" radius="0.033"/>
+        <cylinder length="0.020" radius="0.072"/>
       </geometry>
     </collision>
@@ -63,5 +63,5 @@
     <parent link="base_link"/>
     <child link="wheel_right_link"/>
-    <origin xyz="0.0 -0.144 0.023" rpy="-1.57 0 0"/>
+    <origin xyz="0.0 -0.288 0.023" rpy="-1.57 0 0"/>
     <axis xyz="0 0 1"/>
   </joint>
@@ -70,5 +70,5 @@
       <origin xyz="0 0 0" rpy="1.57 0 0"/>
       <geometry>
-        <mesh filename="package://amazon_robot_description/meshes/wheels/right_tire.stl" scale="0.001 0.001 0.001"/>
+        <mesh filename="package://amazon_robot_description/meshes/wheels/right_tire.stl" scale="0.002 0.002 0.002"/>
       </geometry>
       <material name="dark"/>
@@ -77,5 +77,5 @@
       <origin xyz="0 0 0" rpy="0 0 0"/>
       <geometry>
-        <cylinder length="0.018" radius="0.033"/>
+        <cylinder length="0.020" radius="0.072"/>
       </geometry>
     </collision>
@@ -91,5 +91,5 @@
     <parent link="base_link"/>
     <child link="caster_back_right_link"/>
-    <origin xyz="-0.177 -0.064 -0.004" rpy="-1.57 0 0"/>
+    <origin xyz="-0.268 -0.064 -0.016" rpy="-1.57 0 0"/>
   </joint>
   <link name="caster_back_right_link">
@@ -97,5 +97,5 @@
       <origin xyz="0 0.001 0" rpy="0 0 0"/>
       <geometry>
-        <box size="0.030 0.009 0.020"/>
+        <box size="0.060 0.018 0.040"/>
       </geometry>
     </collision>
@@ -111,5 +111,5 @@
     <parent link="base_link"/>
     <child link="caster_back_left_link"/>
-    <origin xyz="-0.177 0.064 -0.004" rpy="-1.57 0 0"/>
+    <origin xyz="-0.268 0.064 -0.016" rpy="-1.57 0 0"/>
   </joint>
   <link name="caster_back_left_link">
@@ -117,5 +117,5 @@
       <origin xyz="0 0.001 0" rpy="0 0 0"/>
       <geometry>
-        <box size="0.030 0.009 0.020"/>
+        <box size="0.060 0.018 0.040"/>
       </geometry>
     </collision>
@@ -131,5 +131,5 @@
     <parent link="base_link"/>
     <child link="imu_link"/>
-    <origin xyz="0.0 0 0.068" rpy="0 0 0"/>
+    <origin xyz="0.0 0 0.136" rpy="0 0 0"/>
   </joint>
   <link name="imu_link"/>
@@ -137,5 +137,5 @@
     <parent link="base_link"/>
     <child link="base_scan"/>
-    <origin xyz="-0.064 0 0.122" rpy="0 0 0"/>
+    <origin xyz="-0.064 0 0.244" rpy="0 0 0"/>
   </joint>
   <link name="base_scan">
@@ -143,5 +143,5 @@
       <origin xyz="0 0 0.0" rpy="0 0 0"/>
       <geometry>
-        <mesh filename="package://amazon_robot_description/meshes/sensors/lds.stl" scale="0.001 0.001 0.001"/>
+        <mesh filename="package://amazon_robot_description/meshes/sensors/lds.stl" scale="0.002 0.002 0.002"/>
       </geometry>
       <material name="dark"/>
@@ -201,5 +201,5 @@
     <visual>
       <geometry>
-        <box size="0.02 0.02 0.08" />
+        <box size="0.02 0.02 0.10" />
       </geometry>
       <material name="blue"/>
@@ -207,5 +207,5 @@
     <collision>
       <geometry>
-        <box size="0.02 0.02 0.08" />
+        <box size="0.02 0.02 0.10" />
       </geometry>
     </collision>
@@ -221,5 +221,5 @@
     <parent link="base_link" />
     <child link="link_platform_mid" />
-    <origin xyz="-0.08 0 0.10" rpy="0. 0. 0."/>
+    <origin xyz="-0.08 0 0.20" rpy="0. 0. 0."/>
   </joint>
   <link name="lift_link">
@@ -250,10 +250,10 @@
 <!--  </joint>-->
   <joint name="lift_joint" type="prismatic" >
-  <origin xyz="0 0 0.04" rpy="0. 0. 0."/>
+  <origin xyz="0 0 0.16" rpy="0. 0. 0."/>
     <child link="lift_link" />
     <parent link="link_platform_mid" />
     <axis xyz="0 0 1" rpy="0 0 0"/>
-    <limit effort="0.0" lower="0.0" upper="2" velocity="0.005"/>
-    <inertia ixx="0" ixy="0.0" ixz="0" iyy="0" iyz="0" izz="0"/>
+    <limit effort="10000.0" lower="-0.05" upper="0.20" velocity="0.5"/>
+<!--    <inertia ixx="0" ixy="0.0" ixz="1" iyy="0" iyz="0" izz="0"/>-->
   </joint>
 <!--      <joint type="screw" name="lift_joint">-->
@@ -275,5 +275,5 @@
 <!--      <origin xyz="0 0 0" rpy="0 0 0"/>-->
 <!--      <geometry>-->
-<!--        <mesh filename="package://amazon_robot_description/meshes/bases/waffle_base.stl" scale="0.001 0.001 0.001"/>-->
+<!--        <mesh filename="package://amazon_robot_description/meshes/bases/waffle_base.stl" scale="0.002 0.002 0.002"/>-->
 <!--      </geometry>-->
 <!--      <material name="dark"/>-->

Commit message: Simulation: Complete amazon exercise working

File: catkin_workspace/src/amazon_robot_description/urdf/amazon_warehouse_robot.gazebo.xacro (robot description, xacro)
@@ -51,4 +51,10 @@
     <material>Gazebo/FlatBlack</material>
   </gazebo>
+  <gazebo reference="lift_joint">
+    <mu1>20000</mu1>
+    <mu2>20000</mu2>
+    <kp>1000000.0</kp>
+    <material>Gazebo/Red</material>
+  </gazebo>
   <gazebo reference="imu_link">
     <sensor type="imu" name="imu">
@@ -60,4 +66,5 @@
   <gazebo>
     <plugin name="drive_controller" filename="libgazebo_ros_diff_drive.so">
+      <alwaysOn>true</alwaysOn>
       <commandTopic>cmd_vel</commandTopic>
       <odometryTopic>odom</odometryTopic>
@@ -82,4 +89,5 @@
 <!--      <wheelTorque>10</wheelTorque>-->
       <rosDebugLevel>na</rosDebugLevel>
+      <allow_multiple_cmd_vel_publishers>true</allow_multiple_cmd_vel_publishers>
     </plugin>
   </gazebo>

File: catkin_workspace/src/amazon_robot_description/urdf/amazon_warehouse_robot.urdf.xacro (robot description, xacro)
@@ -221,5 +221,5 @@
     <parent link="base_link" />
     <child link="link_platform_mid" />
-    <origin xyz="-0.08 0 0.20" rpy="0. 0. 0."/>
+    <origin xyz="0.0 0 0.20" rpy="0. 0. 0."/>
   </joint>
   <link name="lift_link">
@@ -227,5 +227,5 @@
     <visual>
       <geometry>
-        <box size="0.30 0.20 0.01" />
+        <box size="0.40 0.40 0.01" />
       </geometry>
       <material name="red"/>
@@ -233,5 +233,5 @@
     <collision>
       <geometry>
-        <box size="0.30 0.20 0.01" />
+        <box size="0.40 0.40 0.01" />
       </geometry>
     </collision>
@@ -254,5 +254,5 @@
     <parent link="link_platform_mid" />
     <axis xyz="0 0 1" rpy="0 0 0"/>
-    <limit effort="10000.0" lower="-0.05" upper="0.20" velocity="0.5"/>
+    <limit effort="10000.0" lower="-0.05" upper="0.24" velocity="0.5"/>
 <!--    <inertia ixx="0" ixy="0.0" ixz="1" iyy="0" iyz="0" izz="0"/>-->
   </joint>
